File: Design/MediaRemote/MediaRemote.kicad_pcb (KiCad board)
At the start: 2 copper layers, 100 x 90 mm, 46 parts, among them J1 USB_B, J2 JTAG, J3 LCD Connector, SW1 PEC11R-4020F-S0024, SW2 Cherry MX Green, SW3 Cherry MX Green, SW4 Cherry MX Green, SW5 Cherry MX Green, U1 AZ1117-3.3, U2 STM32F722RETx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

Commit message: Updated PCB
Parts:
- moved C3 5.51 mm to (116.2, 63.8), turned to 270 degrees
- moved C4 5.51 mm to (103.8, 63.8), turned to 270 degrees
- moved R3 2.30 mm to (114.0, 63.8), turned to 90 degrees
- moved R4 2.30 mm to (106.0, 63.8), turned to 90 degrees
- moved R1 1.77 mm to (111.8, 63.8), turned to 270 degrees
- moved R2 1.77 mm to (108.2, 63.8), turned to 270 degrees
- moved C18 1.00 mm to (71.5, 95.0)
- moved C19 1.00 mm to (95.5, 95.0)
- moved R10 1.00 mm to (98.0, 95.0)
- moved R5 1.00 mm to (76.5, 95.0)
- moved R6 1.00 mm to (100.5, 95.0)
- moved R9 1.00 mm to (74.0, 95.0)
- moved SW2 1.00 mm to (76.5, 101.9)
- moved SW3 1.00 mm to (100.5, 101.9)
- moved C21 0.47 mm to (143.5, 94.9)
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Routing:
- net Net-(R2-Pad2): track 6.00 -> 5.31 mm
- net Net-(R1-Pad2): track 6.00 -> 5.31 mm
Other:
- outline, holes or cut-outs redrawn
